File: pinky-8.sch (KiCad schematic (older format))
At the start: 23 parts, among them P1 USB_B, P2 PERIPHERAL A, P3 PERIPHERAL B, P4 2x3 HEADER, SW1 SW_Push_Dual, U1 W65C02S, U2 74AC00, U3 AS6C62256, U4 DS1813, U5 GLS29EE010, U6 W65C22S, X1 MXO45

Commit message: Updating to Rev B spec.
Parts:
- removed P4: 2x3 HEADER, Pin_Headers:Pin_Header_Straight_2x03_Pitch2.54mm, symbol CONN_02X03
- removed R1: 3.3K, Resistors_THT:R_Axial_DIN0204_L3.6mm_D1.6mm_P7.62mm_Horizontal, symbol R
- added P1, P10, P11, P13, P14, P15, P17, P2, P3, P4, P5, P6: CONN_01X01, Wire_Pads:SolderWirePad_single_0-8mmDrill, symbol CONN_01X01
- added P7, P8, P9: CONN_01X03, Pin_Headers:Pin_Header_Straight_1x03_Pitch2.54mm, symbol CONN_01X03
- added SW1: SW_Push_Dual, Buttons_Switches_THT:SW_TH_Tactile_Omron_B3F-10xx, symbol SW_Push_Dual
- added U6: DS1813, TO_SOT_Packages_THT:TO-92_Inline_Wide, symbol DS1813
- renumbered C3 to C1, C5 to C2, C6 to C3, C7 to C5, C1 to C6, C2 to C7, P2 to P12, P3 to P16, P1 to P18, R2 to R1, R5 to R2, R4 to R3, SW1 to SW2, U3 to U1, U5 to U2, U1 to U3, U2 to U4, U6 to U5, U4 to U7
Connections:
- net A13: no longer U5.24 (CS1)
- net A14: now also U4.12 (4A), U4.9 (3A); no longer U1.22 (OE#), U2.29 (A14)
- net A15: now also U4.13 (4B), U4.2 (1B), U5.24 (CS1)
- net CLK: now also U4.5 (2B), U5.25 (PHI2)
- net GND: now also P13.1 (P1), P14.1 (P1), P17.1 (P1), P4.1 (P1), P5.1 (P1), P6.1 (P1), SW1.4, U6.3 (GND)
- net RB0: now also U2.29 (A14), P7.2 (P2); no longer U2.3 (A15)
- net RB1: now also U2.3 (A15), P8.2 (P2); no longer U2.2 (A16)
- net VCC: now also R2.2, P1.1 (P1), P10.1 (P1), P11.1 (P1), P15.1 (P1), P2.1 (P1), P3.1 (P1), U6.2 (VCC); no longer R2.1
- net PLDN: now reaches R3.1
- net PLDN: now also P7.3 (P3), P8.3 (P3), P9.3 (P3)
- net ROMSEL#: now reaches U4.11 (4Y)
- net ROMSEL#: now also U2.22 (CE#), U2.24 (OE#)
- net IRQ renamed IRQ#
- removed net PHI2: U3.39 (PHI2o), U4.5 (2B), U5.25 (PHI2)
- net RAMSEL renamed RAMSEL#
- net RAMSEL#: now also U1.22 (OE#)
- removed net ROMSEL: U2.22 (CE#), U2.24 (OE#), U4.3 (1Y), U4.4 (2A), U4.9 (3A)
- net RST renamed RST#
- net RW renamed RW#
- net VIASEL renamed VIASEL#
- new net: R1.2, U3.2 (RDY)
- new net A15#: U4.3 (1Y), U4.4 (2A)
- new net NMI#: SW1.2, U3.6 (NMI#), U6.1 (RST#)
- new net PLUP: P7.1 (P1), P8.1 (P1), P9.1 (P1), R2.1, U3.36 (BE), U3.38 (SO#)
- new net RB2: P9.2 (P2), U2.2 (A16)
Other:
- note added: "8/9/2017"
- note added: "A barebones, 65C02S-based 8-bit microcomputer SBC inspired by Garth Wilson's \n6502 primer (http://wilsonminesco.com/6502primer).\nDesigned for operation at 5Mhz with 32K of addressable RAM\nand eight manually-selectable 16K ROM banks."
- note added: "B"
- note added: "NMI"
- note added: "Static Logic Levels"
- note removed: "6/7/2017"
- note removed: "A"
- note removed: "A barebones, 65C02S-based 8-bit microcomputer SBC building on Garth Wilson's \n6502 primer (http://wilsonminesco.com/6502primer).\nDesigned for operation at 5Mhz with 16K of addressable RAM\nand manually-selectable 32K ROM banks."
- moved on the sheet: C6, R1, R2, R3, X1

Commit message: Fixing a routing error
Connections:
- net A14: now also U5.23 (CS2#); no longer U4.10 (3B), U4.9 (3A)
- net PLDN: now also U4.10 (3B), U4.9 (3A)
- net VIASEL#: no longer names the net of U4.8 (3Y)
- net VIASEL#: no longer U5.23 (CS2#)
- no-connect marks 13 -> 14
Changed lines of the file:
@@
 	8850 4550 8950 4550
 Text Label 8950 4550 0    60   ~ 0
-VIASEL#
+A14
 Wire Wire Line
 	8850 4450 8950 4450
@@
 Text Label 3750 5050 2    60   ~ 0
 RAMSEL#
-Text Label 4650 4500 0    60   ~ 0
-A14
-Text Label 4650 4700 0    60   ~ 0
-VIASEL#
 $Comp
 L C C4
@@
 Text Label 4650 5050 0    60   ~ 0
 ROMSEL#
-Text Label 4650 4600 0    60   ~ 0
-A14
 Text Label 3750 4600 2    60   ~ 0
 A15
@@
 L CONN_01X01 P10
 U 1 1 598E70C0
-P 4900 4550
-F 0 "P10" H 4900 4650 50  0001 C CNN
-F 1 "CONN_01X01" V 5000 4550 50  0001 C CNN
-F 2 "Wire_Pads:SolderWirePad_single_0-8mmDrill" H 4900 4550 50  0001 C CNN
-F 3 "" H 4900 4550 50  0000 C CNN
-	1    4900 4550
+P 4900 4350
+F 0 "P10" H 4900 4450 50  0001 C CNN
+F 1 "CONN_01X01" V 5000 4350 50  0001 C CNN
+F 2 "Wire_Pads:SolderWirePad_single_0-8mmDrill" H 4900 4350 50  0001 C CNN
+F 3 "" H 4900 4350 50  0000 C CNN
+	1    4900 4350
 	-1   0    0    1
 $EndComp
@@
 L CONN_01X01 P13
 U 1 1 598E720F
-P 4900 4900
-F 0 "P13" H 4900 5000 50  0001 C CNN
-F 1 "CONN_01X01" V 5000 4900 50  0001 C CNN
-F 2 "Wire_Pads:SolderWirePad_single_0-8mmDrill" H 4900 4900 50  0001 C CNN
-F 3 "" H 4900 4900 50  0000 C CNN
-	1    4900 4900
+P 4900 5200
+F 0 "P13" H 4900 5300 50  0001 C CNN
+F 1 "CONN_01X01" V 5000 5200 50  0001 C CNN
+F 2 "Wire_Pads:SolderWirePad_single_0-8mmDrill" H 4900 5200 50  0001 C CNN
+F 3 "" H 4900 5200 50  0000 C CNN
+	1    4900 5200
 	-1   0    0    1
 $EndComp
@@
 Connection ~ 3500 5950
 Connection ~ 3700 6250
-Connection ~ 5100 4550
 Wire Wire Line
 	2350 7150 2650 7150
 Connection ~ 2650 7150
+NoConn ~ 4650 4700
+Text Label 4650 4600 0    60   ~ 0
+PLDN
+Text Label 4650 4500 0    60   ~ 0
+PLDN
+Connection ~ 5100 4350
+Connection ~ 5100 5200
 $EndSCHEMATC

Commit message: Updating to latest KiCad format
Parts:
- C1, C2, C3, C4, C5, C6: symbol C -> device:C
- C7: symbol CP -> device:CP
- P1, P10, P11, P13, P14, P15, P17, P2, P3, P4, P5, P6: symbol CONN_01X01 -> conn:CONN_01X01
- P12, P16: symbol CONN_02X07 -> conn:CONN_02X07
- P18: symbol USB_B -> conn:USB_B
- P7, P8, P9: symbol CONN_01X03 -> conn:CONN_01X03
- R1, R2, R3: symbol R -> device:R
- SW1, SW2: symbol SW_Push_Dual -> switches:SW_Push_Dual
- U1: symbol AS6C62256 -> retrocomps:AS6C62256
- U2: symbol GLS29EE010 -> retrocomps:GLS29EE010
- U3: symbol W65C02S -> w65c:W65C02S
- U4: symbol 74HC00_DIP-14 -> retrocomps:74HC00_DIP-14
- U5: symbol W65C22S -> w65c:W65C22S
- U6, U7: symbol DS1813 -> retrocomps:DS1813
- X1: symbol TCXO3 -> Oscillators:TCXO3
